Commit message: feat: 실물 OpenArm 제조 연동 및 각종 트러블 슈팅
- MoveIt, planning scene 동기화, CAN 인터페이스, 컨트롤러 시작을 묶은 실물 OpenArm 제조 launch 흐름 추가
- KDL dynamics, gravity/coriolis 보상 옵션, legacy fallback을 포함한 OpenArm hardware interface 벤더링
- 실물 로봇 제어용 forward joint trajectory bridge 노드와 gravity compensation 노드 추가
- hardware plugin 선택과 forward controller 사용을 위해 OpenArm URDF, ros2_control, controller, gain 설정 갱신
- 핫도그 task preset/launch 동작을 확장하고 Gazebo, MoveIt, 실물 OpenArm, 서비스 연동 실행 문서 갱신

File: src/controller/ddooby_controller/openarm_vendor/openarm_description/urdf/robot/openarm_robot.xacro (robot description, xacro)
@@ -38,4 +38,10 @@
             right_arm_prefix:='right_'
             can_fd:='true'
+            hardware_plugin:='openarm_hardware/OpenArmHW'
+            return_to_zero_on_activate:='false'
+            hold_current_on_activate:='true'
+            enable_gravity_comp:='true'
+            enable_coriolis_comp:='false'
+            gravity_comp_start_delay_sec:='8.0'
             "
             >
@@ -104,5 +110,12 @@
             left_arm_prefix="${left_arm_prefix}"
             right_arm_prefix="${right_arm_prefix}"
-            hand="${hand}"/>
+            hand="${hand}"
+            can_fd="${can_fd}"
+            hardware_plugin="${hardware_plugin}"
+            return_to_zero_on_activate="${return_to_zero_on_activate}"
+            hold_current_on_activate="${hold_current_on_activate}"
+            enable_gravity_comp="${enable_gravity_comp}"
+            enable_coriolis_comp="${enable_coriolis_comp}"
+            gravity_comp_start_delay_sec="${gravity_comp_start_delay_sec}"/>
         </xacro:if>
         <xacro:if value="$(eval hand and ee_type == 'openarm_hand')">
@@ -158,5 +171,11 @@
             hand="${hand}"
             bimanual="false"
-            can_fd="${can_fd}"/>
+            can_fd="${can_fd}"
+            hardware_plugin="${hardware_plugin}"
+            return_to_zero_on_activate="${return_to_zero_on_activate}"
+            hold_current_on_activate="${hold_current_on_activate}"
+            enable_gravity_comp="${enable_gravity_comp}"
+            enable_coriolis_comp="${enable_coriolis_comp}"
+            gravity_comp_start_delay_sec="${gravity_comp_start_delay_sec}"/>
         </xacro:if>
         <xacro:if value="${hand and ee_type == 'openarm_hand'}">

File: src/controller/ddooby_controller/openarm_vendor/openarm_description/urdf/robot/v10.urdf.xacro (robot description, xacro)
@@ -27,4 +27,10 @@
   <xacro:arg name="left_arm_base_rpy" default="-1.5708 0 0" />
   <xacro:arg name="can_fd" default="true" />
+  <xacro:arg name="hardware_plugin" default="openarm_hardware/OpenArmHW" />
+  <xacro:arg name="return_to_zero_on_activate" default="false" />
+  <xacro:arg name="hold_current_on_activate" default="true" />
+  <xacro:arg name="enable_gravity_comp" default="true" />
+  <xacro:arg name="enable_coriolis_comp" default="false" />
+  <xacro:arg name="gravity_comp_start_delay_sec" default="8.0" />
   <xacro:openarm_robot
   arm_type="v10"
@@ -61,4 +67,10 @@
   left_arm_base_rpy="$(arg left_arm_base_rpy)"
   can_fd="$(arg can_fd)"
+  hardware_plugin="$(arg hardware_plugin)"
+  return_to_zero_on_activate="$(arg return_to_zero_on_activate)"
+  hold_current_on_activate="$(arg hold_current_on_activate)"
+  enable_gravity_comp="$(arg enable_gravity_comp)"
+  enable_coriolis_comp="$(arg enable_coriolis_comp)"
+  gravity_comp_start_delay_sec="$(arg gravity_comp_start_delay_sec)"
   />
 </robot>

File: src/controller/ddooby_controller/openarm_vendor/openarm_description/urdf/ros2_control/openarm.bimanual.ros2_control.xacro (robot description, xacro)
@@ -11,5 +11,11 @@
              left_arm_prefix:=^|left_
              right_arm_prefix:=^|right_
-             can_fd:=^|true">
+             can_fd:=^|true
+             hardware_plugin:=^|openarm_hardware/OpenArmHW
+             return_to_zero_on_activate:=^|false
+             hold_current_on_activate:=^|true
+             enable_gravity_comp:=^|true
+             enable_coriolis_comp:=^|false
+             gravity_comp_start_delay_sec:=^|8.0">
     <!-- Left Arm Hardware Interface -->
     <ros2_control name="openarm_left_hardware_interface" type="system">
@@ -22,9 +28,14 @@
           </xacro:if>
           <xacro:unless value="${use_fake_hardware}">
-            <plugin>openarm_hardware/OpenArm_v10HW</plugin>
+            <plugin>${hardware_plugin}</plugin>
             <param name="can_interface">${left_can_interface}</param>
             <param name="arm_prefix">${left_arm_prefix}</param>
             <param name="hand">${hand}</param>
             <param name="can_fd">${can_fd}</param>
+            <param name="return_to_zero_on_activate">${return_to_zero_on_activate}</param>
+            <param name="hold_current_on_activate">${hold_current_on_activate}</param>
+            <param name="enable_gravity_comp">${enable_gravity_comp}</param>
+            <param name="enable_coriolis_comp">${enable_coriolis_comp}</param>
+            <param name="gravity_comp_start_delay_sec">${gravity_comp_start_delay_sec}</param>
             <param name="kp1">${control_gains['joint1']['kp']}</param>
             <param name="kp2">${control_gains['joint2']['kp']}</param>
@@ -63,4 +74,15 @@
         </joint>
       </xacro:macro>
+      <xacro:macro name="configure_gripper_joint" params="joint_name initial_position">
+        <joint name="${joint_name}">
+          <command_interface name="position"/>
+          <state_interface name="position">
+            <param name="initial_value">${initial_position}</param>
+          </state_interface>
+          <state_interface name="velocity">
+            <param name="initial_value">0.0</param>
+          </state_interface>
+        </joint>
+      </xacro:macro>
       <xacro:configure_joint joint_name="openarm_${left_arm_prefix}joint1" initial_position="0.0"/>
       <xacro:configure_joint joint_name="openarm_${left_arm_prefix}joint2" initial_position="0.0"/>
@@ -71,5 +93,5 @@
       <xacro:configure_joint joint_name="openarm_${left_arm_prefix}joint7" initial_position="0.0"/>
       <xacro:if value="${hand}">
-        <xacro:configure_joint joint_name="openarm_${left_arm_prefix}finger_joint1" initial_position="0.0" />
+        <xacro:configure_gripper_joint joint_name="openarm_${left_arm_prefix}finger_joint1" initial_position="0.0" />
       </xacro:if>
     </ros2_control>
@@ -84,9 +106,14 @@
           </xacro:if>
           <xacro:unless value="${use_fake_hardware}">
-            <plugin>openarm_hardware/OpenArm_v10HW</plugin>
+            <plugin>${hardware_plugin}</plugin>
             <param name="can_interface">${right_can_interface}</param>
             <param name="arm_prefix">${right_arm_prefix}</param>
             <param name="hand">${hand}</param>
             <param name="can_fd">${can_fd}</param>
+            <param name="return_to_zero_on_activate">${return_to_zero_on_activate}</param>
+            <param name="hold_current_on_activate">${hold_current_on_activate}</param>
+            <param name="enable_gravity_comp">${enable_gravity_comp}</param>
+            <param name="enable_coriolis_comp">${enable_coriolis_comp}</param>
+            <param name="gravity_comp_start_delay_sec">${gravity_comp_start_delay_sec}</param>
             <param name="kp1">${control_gains['joint1']['kp']}</param>
             <param name="kp2">${control_gains['joint2']['kp']}</param>
@@ -117,5 +144,5 @@
       <xacro:configure_joint joint_name="openarm_${right_arm_prefix}joint7" initial_position="0.0"/>
       <xacro:if value="${hand}">
-        <xacro:configure_joint joint_name="openarm_${right_arm_prefix}finger_joint1" initial_position="0.0" />
+        <xacro:configure_gripper_joint joint_name="openarm_${right_arm_prefix}finger_joint1" initial_position="0.0" />
       </xacro:if>
     </ros2_control>

File: src/controller/ddooby_controller/openarm_vendor/openarm_description/urdf/ros2_control/openarm.ros2_control.xacro (robot description, xacro)
@@ -11,5 +11,11 @@
              arm_prefix:=''
              bimanual:=false
-             can_fd:=^|true">
+             can_fd:=^|true
+             hardware_plugin:=^|openarm_hardware/OpenArmHW
+             return_to_zero_on_activate:=^|false
+             hold_current_on_activate:=^|true
+             enable_gravity_comp:=^|true
+             enable_coriolis_comp:=^|false
+             gravity_comp_start_delay_sec:=^|8.0">
     <ros2_control name="openarm_hardware_interface" type="system">
         <hardware>
@@ -22,9 +28,14 @@
           </xacro:if>
           <xacro:if value="${use_fake_hardware == 0}">
-            <plugin>openarm_hardware/OpenArm_${arm_type}HW</plugin>
+            <plugin>${hardware_plugin}</plugin>
             <param name="can_interface">${can_interface}</param>
             <param name="arm_prefix">${arm_prefix}</param>
             <param name="hand">${hand}</param>
             <param name="can_fd">${can_fd}</param>
+            <param name="return_to_zero_on_activate">${return_to_zero_on_activate}</param>
+            <param name="hold_current_on_activate">${hold_current_on_activate}</param>
+            <param name="enable_gravity_comp">${enable_gravity_comp}</param>
+            <param name="enable_coriolis_comp">${enable_coriolis_comp}</param>
+            <param name="gravity_comp_start_delay_sec">${gravity_comp_start_delay_sec}</param>
             <param name="kp1">${control_gains['joint1']['kp']}</param>
             <param name="kp2">${control_gains['joint2']['kp']}</param>
@@ -68,4 +79,15 @@
         </joint>
       </xacro:macro>
+      <xacro:macro name="configure_gripper_joint" params="joint_name initial_position">
+        <joint name="${joint_name}">
+          <command_interface name="position"/>
+          <state_interface name="position">
+            <param name="initial_value">${initial_position}</param>
+          </state_interface>
+          <state_interface name="velocity">
+            <param name="initial_value">0.0</param>
+          </state_interface>
+        </joint>
+      </xacro:macro>
       <xacro:configure_joint joint_name="openarm_${arm_prefix}joint1" initial_position="0.0"/>
       <xacro:configure_joint joint_name="openarm_${arm_prefix}joint2" initial_position="0.0"/>
@@ -76,5 +98,5 @@
       <xacro:configure_joint joint_name="openarm_${arm_prefix}joint7" initial_position="0.0"/>
       <xacro:if value="${hand}">
-        <xacro:configure_joint joint_name="openarm_${arm_prefix}finger_joint1" initial_position="0.0" />
+        <xacro:configure_gripper_joint joint_name="openarm_${arm_prefix}finger_joint1" initial_position="0.0" />
       </xacro:if>
     </ros2_control>
