Commit message: fix: 실물 그리퍼 형상 반영 및 핫도그 제조 튜닝 갱신
- 실물 그리퍼 DAE 메시를 직접 모델링 및 추가하고 OpenArm hand URDF 참조를 새 메시로 변경
- 소시지, 소시지 트레이, 소시지 트레이 스탠드 Gazebo 모델 추가
- 기존 트레이 스탠드 에셋을 빵 트레이 스탠드로 변경하고 제조 월드 배치 갱신
- 핫도그 작업 pose, 그리퍼 목표값, TCP 오프셋, 플래닝 재시도 동작 튜닝
- Cartesian 및 stage pose 이동에 최소 trajectory duration 처리 추가

File: src/controller/ddooby_controller/openarm_vendor/openarm_description/urdf/ee/openarm_hand.xacro (robot description, xacro)
@@ -29,5 +29,5 @@
         <xacro:openarm-ee-kinematics-link config="${ee_kinematics_link}" name="left_finger" />
         <geometry>
-          <mesh filename="package://${description_pkg}/meshes/ee/${ee_type}/visual/finger.dae" scale="0.001 0.001 0.001"/>
+          <mesh filename="package://${description_pkg}/meshes/ee/${ee_type}/visual/gripper.dae" scale="0.001 0.001 0.001"/>
         </geometry>
       </visual>
@@ -35,5 +35,5 @@
         <xacro:openarm-ee-kinematics-link config="${ee_kinematics_link}" name="left_finger" />
         <geometry>
-          <mesh filename="package://${description_pkg}/meshes/ee/${ee_type}/collision/finger.stl" scale="0.001 0.001 0.001" />
+          <mesh filename="package://${description_pkg}/meshes/ee/${ee_type}/collision/gripper.dae" scale="0.001 0.001 0.001" />
         </geometry>
       </collision>
@@ -44,5 +44,5 @@
         <xacro:openarm-ee-kinematics-link config="${ee_kinematics_link}" name="right_finger" />
         <geometry>
-          <mesh filename="package://${description_pkg}/meshes/ee/${ee_type}/visual/finger.dae" scale="0.001 -0.001 0.001"/>
+          <mesh filename="package://${description_pkg}/meshes/ee/${ee_type}/visual/gripper.dae" scale="0.001 -0.001 0.001"/>
         </geometry>
       </visual>
@@ -50,5 +50,5 @@
         <xacro:openarm-ee-kinematics-link config="${ee_kinematics_link}" name="right_finger" />
         <geometry>
-          <mesh filename="package://${description_pkg}/meshes/ee/${ee_type}/collision/finger.stl" scale="0.001 -0.001 0.001" />
+          <mesh filename="package://${description_pkg}/meshes/ee/${ee_type}/collision/gripper.dae" scale="0.001 -0.001 0.001" />
         </geometry>
       </collision>

File: src/controller/ddooby_controller/openarm_vendor/openarm_description/urdf/ee/openarm_hand_arguments.xacro (robot description, xacro)
@@ -8,5 +8,5 @@
   <xacro:arg name="rpy_ee" default= "0 0 0" />
   <!-- Position offset between ee frame and tcp frame -->
-  <xacro:arg name="tcp_xyz" default="0 -0.0 0.08" />
+  <xacro:arg name="tcp_xyz" default="0 -0.0 0.13" />
   <!-- Rotation offset between ee frame and tcp frame -->
   <xacro:arg name="tcp_rpy" default="0 0 0" />
